Commit message: Fix really bad problems with drifting but not done yet

File: muse_ws/src/state_estimator/urdfs/go1.urdf (robot description, URDF)
Before this commit: robot go1, 46 links, 45 joints
Links:
- removed link FL_calf_rotor
- removed link FL_hip_rotor
- removed link FL_thigh_rotor
- removed link FR_calf_rotor
- removed link FR_hip_rotor
- removed link FR_thigh_rotor
- removed link RL_calf_rotor
- removed link RL_hip_rotor
- removed link RL_thigh_rotor
- removed link RR_calf_rotor
- removed link RR_hip_rotor
- removed link RR_thigh_rotor
- removed link base
- removed link camera_chin
- removed link camera_face
- removed link camera_laserscan_link_left
- removed link camera_laserscan_link_right
- removed link camera_left
- removed link camera_optical_chin
- removed link camera_optical_face
- removed link camera_optical_left
- removed link camera_optical_rearDown
- removed link camera_optical_right
- removed link camera_rearDown
- removed link camera_right
- removed link imu_link
- removed link trunk
- removed link ultraSound_face
- removed link ultraSound_left
- removed link ultraSound_right
- added link FL_calflower; collision cylinder length=0.065 radius=0.011
- added link FL_calflower1; collision cylinder length=0.03 radius=0.0155
- added link FR_calflower; collision cylinder length=0.065 radius=0.011
- added link FR_calflower1; collision cylinder length=0.03 radius=0.0155
- added link Head_lower, mass 0.001; collision sphere radius=0.047
- added link Head_upper, mass 0.001; collision cylinder length=0.09 radius=0.05
- added link RL_calflower; collision cylinder length=0.065 radius=0.011
- added link RL_calflower1; collision cylinder length=0.03 radius=0.0155
- added link RR_calflower; collision cylinder length=0.065 radius=0.011
- added link RR_calflower1; collision cylinder length=0.03 radius=0.0155
- added link base_link, mass 6.921; collision box size=0.3762 0.0935 0.114; visual mesh filename=package://go2_description/dae/base.dae
- added link imu, mass 0
- added link radar, mass 0
- link FL_calf: mass 0.135862 -> 0.154; geometry collision cylinder length=0.12 radius=0.012; visual mesh filename=package://go2_description/dae/calf.dae
- link FL_foot: mass 0.06 -> 0.04; geometry collision sphere radius=0.022; visual mesh filename=package://go2_description/dae/foot.dae
- link FL_hip: mass 0.591 -> 0.678; geometry collision cylinder length=0.04 radius=0.046; visual mesh filename=package://go2_description/dae/hip.dae
- link FL_thigh: mass 0.92 -> 1.152; geometry collision box size=0.213 0.0245 0.034; visual mesh filename=package://go2_description/dae/thigh.dae
- link FR_calf: mass 0.135862 -> 0.154; geometry collision cylinder length=0.12 radius=0.013; visual mesh filename=package://go2_description/dae/calf_mirror.dae
- link FR_foot: mass 0.06 -> 0.04; geometry collision sphere radius=0.022; visual mesh filename=package://go2_description/dae/foot.dae
- link FR_hip: mass 0.591 -> 0.678; geometry collision cylinder length=0.04 radius=0.046; visual mesh filename=package://go2_description/dae/hip.dae
- link FR_thigh: mass 0.92 -> 1.152; geometry collision box size=0.213 0.0245 0.034; visual mesh filename=package://go2_description/dae/thigh_mirror.dae
- link RL_calf: mass 0.135862 -> 0.154; geometry collision cylinder length=0.12 radius=0.013; visual mesh filename=package://go2_description/dae/calf.dae
- link RL_foot: mass 0.06 -> 0.04; geometry collision sphere radius=0.022; visual mesh filename=package://go2_description/dae/foot.dae
- link RL_hip: mass 0.591 -> 0.678; geometry collision cylinder length=0.04 radius=0.046; visual mesh filename=package://go2_description/dae/hip.dae
- link RL_thigh: mass 0.92 -> 1.152; geometry collision box size=0.213 0.0245 0.034; visual mesh filename=package://go2_description/dae/thigh.dae
- link RR_calf: mass 0.135862 -> 0.154; geometry collision cylinder length=0.12 radius=0.013; visual mesh filename=package://go2_description/dae/calf_mirror.dae
- link RR_foot: mass 0.06 -> 0.04; geometry collision sphere radius=0.022; visual mesh filename=package://go2_description/dae/foot.dae
- link RR_hip: mass 0.591 -> 0.678; geometry collision cylinder length=0.04 radius=0.046; visual mesh filename=package://go2_description/dae/hip.dae
- link RR_thigh: mass 0.92 -> 1.152; geometry collision box size=0.213 0.0245 0.034; visual mesh filename=package://go2_description/dae/thigh_mirror.dae
Joints:
- removed joint FL_calf_rotor_joint
- removed joint FL_foot_fixed
- removed joint FL_hip_rotor_joint
- removed joint FL_thigh_rotor_joint
- removed joint FR_calf_rotor_joint
- removed joint FR_foot_fixed
- removed joint FR_hip_rotor_joint
- removed joint FR_thigh_rotor_joint
- removed joint RL_calf_rotor_joint
- removed joint RL_foot_fixed
- removed joint RL_hip_rotor_joint
- removed joint RL_thigh_rotor_joint
- removed joint RR_calf_rotor_joint
- removed joint RR_foot_fixed
- removed joint RR_hip_rotor_joint
- removed joint RR_thigh_rotor_joint
- removed joint camera_joint_chin
- removed joint camera_joint_face
- removed joint camera_joint_left
- removed joint camera_joint_rearDown
- removed joint camera_joint_right
- removed joint camera_laserscan_joint_left
- removed joint camera_laserscan_joint_right
- removed joint camera_optical_joint_chin
- removed joint camera_optical_joint_face
- removed joint camera_optical_joint_left
- removed joint camera_optical_joint_rearDown
- removed joint camera_optical_joint_right
- removed joint floating_base
- removed joint ultraSound_joint_face
- removed joint ultraSound_joint_left
- removed joint ultraSound_joint_right
- added joint FL_calflower1_joint: type fixed, parent FL_calflower, child FL_calflower1, origin xyz=-0.01 0 -0.04 rpy=0 0.48 0, axis 0 0 0
- added joint FL_calflower_joint: type fixed, parent FL_calf, child FL_calflower, origin xyz=0.020 0 -0.148 rpy=0 0.05 0, axis 0 0 0
- added joint FL_foot_joint: type fixed, parent FL_calf, child FL_foot, origin xyz=0 0 -0.213 rpy=0 0 0, axis 0 0 0
- added joint FR_calflower1_joint: type fixed, parent FR_calflower, child FR_calflower1, origin xyz=-0.01 0 -0.04 rpy=0 0.48 0, axis 0 0 0
- added joint FR_calflower_joint: type fixed, parent FR_calf, child FR_calflower, origin xyz=0.020 0 -0.148 rpy=0 0.05 0, axis 0 0 0
- added joint FR_foot_joint: type fixed, parent FR_calf, child FR_foot, origin xyz=0 0 -0.213 rpy=0 0 0, axis 0 0 0
- added joint Head_lower_joint: type fixed, parent Head_upper, child Head_lower, origin xyz=0.008 0 -0.07 rpy=0 0 0, axis 0 0 0
- added joint Head_upper_joint: type fixed, parent base_link, child Head_upper, origin xyz=0.285 0 0.01 rpy=0 0 0, axis 0 0 0
- added joint RL_calflower1_joint: type fixed, parent RL_calflower, child RL_calflower1, origin xyz=-0.01 0 -0.04 rpy=0 0.48 0, axis 0 0 0
- added joint RL_calflower_joint: type fixed, parent RL_calf, child RL_calflower, origin xyz=0.020 0 -0.148 rpy=0 0.05 0, axis 0 0 0
- added joint RL_foot_joint: type fixed, parent RL_calf, child RL_foot, origin xyz=0 0 -0.213 rpy=0 0 0, axis 0 0 0
- added joint RR_calflower1_joint: type fixed, parent RR_calflower, child RR_calflower1, origin xyz=-0.01 0 -0.04 rpy=0 0.48 0, axis 0 0 0
- added joint RR_calflower_joint: type fixed, parent RR_calf, child RR_calflower, origin xyz=0.020 0 -0.148 rpy=0 0.05 0, axis 0 0 0
- added joint RR_foot_joint: type fixed, parent RR_calf, child RR_foot, origin xyz=0 0 -0.213 rpy=0 0 0, axis 0 0 0
- added joint radar_joint: type fixed, parent base_link, child radar, origin xyz=0.28945 0 -0.046825 rpy=0 2.8782 0, axis 0 0 0
- joint FL_calf_joint: limit lower=-2.818 upper=-0.888 effort=35.55 velocity=20.06 -> lower=-2.7227 upper=-0.83776 effort=45.43 velocity=15.70
- joint FL_hip_joint: limit lower=-0.863 upper=0.863 effort=23.7 velocity=30.1 -> lower=-1.0472 upper=1.0472 effort=23.7 velocity=30.1; origin xyz=0.1881 0.04675 0 rpy=0 0 0 -> xyz=0.1934 0.0465 0 rpy=0 0 0; parent trunk -> base_link
- joint FL_thigh_joint: limit lower=-0.686 upper=4.501 effort=23.7 velocity=30.1 -> lower=-1.5708 upper=3.4907 effort=23.7 velocity=30.1; origin xyz=0 0.08 0 rpy=0 0 0 -> xyz=0 0.0955 0 rpy=0 0 0
- joint FR_calf_joint: limit lower=-2.818 upper=-0.888 effort=35.55 velocity=20.06 -> lower=-2.7227 upper=-0.83776 effort=45.43 velocity=15.70
- joint FR_hip_joint: limit lower=-0.863 upper=0.863 effort=23.7 velocity=30.1 -> lower=-1.0472 upper=1.0472 effort=23.7 velocity=30.1; origin xyz=0.1881 -0.04675 0 rpy=0 0 0 -> xyz=0.1934 -0.0465 0 rpy=0 0 0; parent trunk -> base_link
- joint FR_thigh_joint: limit lower=-0.686 upper=4.501 effort=23.7 velocity=30.1 -> lower=-1.5708 upper=3.4907 effort=23.7 velocity=30.1; origin xyz=0 -0.08 0 rpy=0 0 0 -> xyz=0 -0.0955 0 rpy=0 0 0
- joint RL_calf_joint: limit lower=-2.818 upper=-0.888 effort=35.55 velocity=20.06 -> lower=-2.7227 upper=-0.83776 effort=45.43 velocity=15.70
- joint RL_hip_joint: limit lower=-0.863 upper=0.863 effort=23.7 velocity=30.1 -> lower=-1.0472 upper=1.0472 effort=23.7 velocity=30.1; origin xyz=-0.1881 0.04675 0 rpy=0 0 0 -> xyz=-0.1934 0.0465 0 rpy=0 0 0; parent trunk -> base_link
- joint RL_thigh_joint: limit lower=-0.686 upper=4.501 effort=23.7 velocity=30.1 -> lower=-0.5236 upper=4.5379 effort=23.7 velocity=30.1; origin xyz=0 0.08 0 rpy=0 0 0 -> xyz=0 0.0955 0 rpy=0 0 0
- joint RR_calf_joint: limit lower=-2.818 upper=-0.888 effort=35.55 velocity=20.06 -> lower=-2.7227 upper=-0.83776 effort=45.43 velocity=15.70
- joint RR_hip_joint: limit lower=-0.863 upper=0.863 effort=23.7 velocity=30.1 -> lower=-1.0472 upper=1.0472 effort=23.7 velocity=30.1; origin xyz=-0.1881 -0.04675 0 rpy=0 0 0 -> xyz=-0.1934 -0.0465 0 rpy=0 0 0; parent trunk -> base_link
- joint RR_thigh_joint: limit lower=-0.686 upper=4.501 effort=23.7 velocity=30.1 -> lower=-0.5236 upper=4.5379 effort=23.7 velocity=30.1; origin xyz=0 -0.08 0 rpy=0 0 0 -> xyz=0 -0.0955 0 rpy=0 0 0
- joint imu_joint: axis (none) -> 0 0 0; child imu_link -> imu; origin xyz=-0.01592 -0.06659 -0.00617 rpy=0 0 0 -> xyz=-0.02557 0 0.04232 rpy=0 0 0; parent trunk -> base_link
